Commit message: Last update

File: src/krotic_description/urdf/krotic.xacro (robot description, xacro)
@@ -98,5 +98,5 @@
 	</link>
 	<joint name="camera_fixed" type="fixed">
-		<origin xyz="0.2 0 0.1" rpy="0 0 0"/>
+		<origin xyz="0.18 0 0.1" rpy="0 0 0"/>
 		<parent link="base_link"/>
 		<child link="camera"/>
