Commit message: Last changes to the model

File: src/krotic_description/urdf/krotic.urdf (robot description, URDF)
Before this commit: robot krotic, 7 links, 6 joints
Links:
- added link light_sensor, mass 1e-5; collision box size=0.01 0.01 0.01; visual box size=0.01 0.01 0.01
- link left_wheel: geometry collision cylinder length=0.03 radius=0.12; visual cylinder length=0.03 radius=0.12
- link right_wheel: geometry collision cylinder length=0.03 radius=0.12; visual cylinder length=0.03 radius=0.12
Joints:
- added joint light_sensor_joint: type fixed, parent base_link, child light_sensor, origin xyz=0.2 0 0.07 rpy=0 0 0, axis 0 1 0
- joint camera_fixed: origin xyz=0.1 0.1 0.17 rpy=0 0 0 -> xyz=0.18 0 0.1 rpy=0 0 0
- joint sonar_joint: origin xyz=0.2 0 0.10 rpy=0 0 0 -> xyz=0.2 0 0.05 rpy=0 0 0

File: src/krotic_description/urdf/krotic.xacro (robot description, xacro)
@@ -143,4 +143,31 @@
 		<child link="base_sonar"/>
 	</joint>
+	<!-- Light Sensor definition -->
+	<link name="light_sensor">
+		<collision>
+			<origin xyz="0 0 0" rpy="0 0 0"/>
+			<geometry>
+				<box size="0.01 0.01 0.01"/>
+			</geometry>
+		</collision>
+		<visual>
+			<origin xyz="0 0 0" rpy="0 0 0"/>
+			<geometry>
+				<box size="0.01 0.01 0.01"/>
+			</geometry>
+		</visual>
+		<inertial>
+			<mass value="1e-5"/>
+			<origin xyz="0 0 0" rpy="0 0 0"/>
+			<inertia ixx="1e-6" ixy="0" ixz="0" iyy="1e-6" iyz="0" izz="1e-6"/>
+		</inertial>
+	</link>
+	<!-- Create a joint between the sensor and the chassis of the robot -->
+	<joint name="light_sensor_joint" type="fixed">
+		<axis xyz="0 1 0" />
+		<origin rpy="0 0 0" xyz="0.2 0 0.07"/>
+		<parent link="base_link"/>
+		<child link="light_sensor"/>
+	</joint>
 	<!-- End of the robot definition -->
 </robot>
